Commit message: Moved to ros2 jazzy

File: mujoco_ws/src/robotx_description/urdf/robotx_position_compiled.urdf (robot description, URDF)
Before this commit: robot dofbot, 13 links, 12 joints
Joints:
- joint joint1: limit lower=-1.5707963267948966 upper=1.5707963267948966 effort=100 velocity=100.0 -> lower=-2 upper=2 effort=1.0 velocity=10.0
- joint joint2: limit lower=-1.5707963267948966 upper=1.5707963267948966 effort=100 velocity=100.0 -> lower=-2 upper=2 effort=1.0 velocity=10.0
- joint joint3: limit lower=-1.5707963267948966 upper=1.5707963267948966 effort=100 velocity=100.0 -> lower=-2 upper=2 effort=1.0 velocity=10.0
- joint joint4: limit lower=-1.5707963267948966 upper=1.5707963267948966 effort=100 velocity=100.0 -> lower=-2 upper=2 effort=1.0 velocity=10.0
- joint joint5: limit lower=-1.5707963267948966 upper=1.5707963267948966 effort=100 velocity=100.0 -> lower=-2 upper=2 effort=1.0 velocity=10.0
- joint joint5a1: limit lower=-1.5707963267948966 upper=1.5707963267948966 effort=100 velocity=100.0 -> lower=-2 upper=2 effort=1.0 velocity=10.0
- joint joint5a2: limit lower=-1.5707963267948966 upper=1.5707963267948966 effort=100 velocity=100.0 -> lower=-2 upper=2 effort=1.0 velocity=10.0
- joint joint5a3: limit lower=-1.5707963267948966 upper=1.5707963267948966 effort=100 velocity=100.0 -> lower=-2 upper=2 effort=1.0 velocity=10.0
- joint joint5b1: limit lower=-1.5707963267948966 upper=1.5707963267948966 effort=100 velocity=100.0 -> lower=-2 upper=2 effort=1.0 velocity=10.0
- joint joint5b2: limit lower=-1.5707963267948966 upper=1.5707963267948966 effort=100 velocity=100.0 -> lower=-2 upper=2 effort=1.0 velocity=10.0
- joint joint5b3: limit lower=-1.5707963267948966 upper=1.5707963267948966 effort=100 velocity=100.0 -> lower=-2 upper=2 effort=1.0 velocity=10.0
